File: hdw/CH340G/CH340.kicad_sch (KiCad schematic)
At the start: 12 parts, among them J1 USB_A, J2 Serial Connector, U1 CH340C

Commit message: upgrade pcb to use USB C 2.0
Parts:
- removed D1: POWER, Library:L1206, symbol Device:LED
- removed H1, H2: MountingHole, MountingHole:MountingHole_2.2mm_M2_DIN965, symbol Mechanical:MountingHole
- removed J1: USB_A, Library:USB_Micro-B, symbol Connector:USB_A
- removed J2: Serial Connector, Connector_PinHeader_2.54mm:PinHeader_1x05_P2.54mm_Vertical, symbol Connector_Generic:Conn_01x05
- removed R1: 1K, Library:R1206, symbol Device:R
- added J1: Conn_01x06, Connector_PinHeader_2.54mm:PinHeader_1x06_P2.54mm_Vertical, symbol Connector_Generic:Conn_01x06
- added P1: USB_C_Plug_USB2.0, Library:TH_USB_C, symbol Connector:USB_C_Plug_USB2.0
Connections:
- net D+: now also P1.A6 (D+)
- net D-: now also P1.A7 (D-)
- net GND: now also J1.2 (Pin_2), P1.A1 (GND), P1.A12 (GND), P1.B1 (GND), P1.B12 (GND)
- net RST: now also J1.5 (Pin_5)
- net RX: now also J1.4 (Pin_4)
- net TX: now also J1.3 (Pin_3)
- net V3: now also J1.1 (Pin_1)
- net VBUS: now also P1.A4 (VBUS), P1.A9 (VBUS), P1.B4 (VBUS), P1.B9 (VBUS)
- net VCC: now also J1.6 (Pin_6)
- no-connect marks 7 -> 9
Other:
- moved on the sheet: C1, C2, C5, D3, F1, U1

Commit message: wip
Parts:
- removed F1: Polyfuse, Library:F1206, symbol Device:Polyfuse
- removed J1: Conn_01x06, Connector_PinHeader_2.54mm:PinHeader_1x06_P2.54mm_Vertical, symbol Connector_Generic:Conn_01x06
- removed P1: USB_C_Plug_USB2.0, Library:TH_USB_C, symbol Connector:USB_C_Plug_USB2.0
- added H1, H2, H3, H4: MountingHole, MountingHole:MountingHole_3.2mm_M3, symbol Mechanical:MountingHole
- added J1: Conn_01x07, Library:PinHeader_1x07_P2.54mm, symbol Connector_Generic:Conn_01x07
- added P1: USB_C_Receptacle_USB2.0, Library:TH_USB_C, symbol Connector:USB_C_Receptacle_USB2.0
- D1: renamed from D3; footprint Library:D1206 -> Library:SMA_DO_214AC
- renumbered C5 to C3
Connections:
- net RST is gone; now on net RTS: C2.2
- net D+: now also P1.A6 (D+), P1.B6 (D+)
- net D-: now also P1.A7 (D-), P1.B7 (D-)
- net DTR: now also J1.1 (Pin_1)
- net GND: now also J1.6 (Pin_6), P1.A1 (GND), P1.A12 (GND), P1.B1 (GND), P1.B12 (GND), P1.S1 (SHIELD)
- net RX: now also J1.4 (Pin_4)
- net TX: now also J1.5 (Pin_5)
- net V3: now also J1.3 (Pin_3)
- net VBUS: now also P1.A4 (VBUS), P1.A9 (VBUS), P1.B4 (VBUS), P1.B9 (VBUS)
- net VCC: now also D1.1 (K), J1.7 (Pin_7)
- net RTS: now reaches U1.14 (~{RTS})
- net RTS: now also J1.2 (Pin_2)
Other:
- moved on the sheet: D1
