File: hdw/minimal/minimal.kicad_sch (KiCad schematic)
At the start: 5 parts, among them P1 USB_C_Plug_USB2.0, U2 CH340C

Commit message: Save changes at: 1752950752
Parts:
- renumbered C4 to C1, C4 to C2, C4 to C3, U2 to U1
Connections:
- net at U1.5 (UD+): now also P1.A6 (D+); no longer P1.A7 (D-)
- net at U1.6 (UD-): now also P1.A7 (D-); no longer P1.A6 (D+)
Other:
- moved on the sheet: C3, P1
